Commit message: 更新urdf,失败

File: iiwa_tool_description/urdf/iiwa_tool.urdf.xacro (robot description, xacro)
@@ -1,5 +1,5 @@
 <?xml version="1.0"?>
 <!-- Here we define the robot, we named it "iiwa_tool" -->
-<robot xmlns:xacro="http://www.ros.org/wiki/xacro" name="iiwa_tool">
+<robot xmlns:xacro="http://www.ros.org/wiki/xacro" name="Toolone">
   <!-- Import Rviz colors -->
   <xacro:include filename="$(find iiwa_description)/urdf/materials.xacro" />
@@ -54,8 +54,8 @@
   <joint name="tool_tip_joint" type="fixed">
     <parent link="tool_link" />
-    <child link = "tool_link_ee" />
+    <child link = "Toolone_link_ee" />
     <origin xyz="${tool_link_offset}" rpy="0 0 0" />
   </joint>
   <!--  The TCP frame is here defined -->
-  <link name="tool_link_ee"/>
+  <link name="Toolone_link_ee"/>
 </robot>
